File: 3x5_3/dilemma.kicad_sch (KiCad schematic)
At the start: 250 parts, among them J1 USB_C_Receptacle_USB2.0, J102 NA_serial, J105 NA_Conn_01x04_Female, J113 Cirque, J3 NA_GC9A01, J4 Conn_01x05, J5 NA_Conn_01x02, J5001 USB_C_Receptacle_USB2.0, J5002 NA_Conn_01x02, J5003 NA_serial, J5004 NA_GC9A01, J5005 NA_Conn_01x04_Female, J5007 Cirque, J5008 Conn_01x05, J5009 Conn_01x05, J5010 Conn_01x05, SW1 SW_Push, SW101 NA_SW_Push, SW102 NA_SW_Push, SW103 NA_SW_Push, SW104 NA_SW_Push, SW105 NA_SW_Push, SW106 NA_SW_Push, SW107 NA_SW_Push, SW108 NA_SW_Push, SW109 NA_SW_Push, SW112 NA_SW_Push, SW113 NA_SW_Push, SW114 NA_SW_Push, SW115 NA_SW_Push, SW116 NA_SW_Push, SW117 NA_SW_Push, SW118 NA_SW_Push, SW119 NA_SW_Push, SW3001 NA_SW_Push, SW3002 NA_RotaryEncoder_Switch, SW5001 SW_Push, SW5002 NA_SW_Push, SW5003 NA_SW_Push, SW5004 NA_SW_Push, SW5005 NA_SW_Push, SW5006 NA_SW_Push, SW5007 NA_SW_Push, SW5008 NA_SW_Push, SW5009 NA_SW_Push, SW5010 NA_SW_Push, SW5011 NA_SW_Push, SW5012 NA_SW_Push, SW5013 NA_SW_Push, SW5014 NA_SW_Push, SW5015 NA_SW_Push, SW5016 NA_SW_Push, SW5017 NA_SW_Push, SW5018 NA_SW_Push, SW5019 NA_SW_Push, SW5020 NA_RotaryEncoder_Switch, SW5021 SW_SPST, SW5022 SW_SPST, U1 RP2040, U2 W25Q128JVS, U3 XC6210B332MR-G, U4 USBLC6-2P6, U5001 XC6210B332MR-G, U5002 RP2040, U5003 USBLC6-2P6, U5004 W25Q128JVS, U5005 USBLC6-2P6, U5006 USBLC6-2P6, Y1 Crystal_GND24, Y5001 Crystal_GND24

Commit message: 3x5_3 right side layout
Parts:
- removed C1, C2: 1µ, Capacitor_SMD:C_0603_1608Metric, symbol Device:C
- removed C10, C11, C12, C13, C14, C7, C8, C9: 100n, Capacitor_SMD:C_0402_1005Metric, symbol Device:C
- removed C3, C4: 15p, Capacitor_SMD:C_0402_1005Metric, symbol Device:C
- removed C5, C5015, C5017, C6: 1µ, Capacitor_SMD:C_0402_1005Metric, symbol Device:C
- removed D1: LED, LED_SMD:LED_0402_1005Metric, symbol Device:LED
- removed D11, D12, D15, D16, D18, D19, D21, D22, D24, D25, D27, D28, D3, D4, D5, D7, D8, D9: SK6805-EC15, 0xB2_drawings:LED_SK6805-EC15_1.5x1.5mm_P0.6mm_handsolder(1), symbol sk6805-ec15:SK6805-EC15
- removed D2: B5817, Diode_SMD:D_SOD-323, symbol Device:D_Schottky
- removed D30, D31, D32, D33, D34, D35, D36, D37: D_CC, local-libraries:SOT-323_SC-70, symbol Device:D_Dual_CommonCathode_AAK
- removed D5031, D5032, D5033, D5034, D5035, D5036, D5037, D5038, D5039, D5040, D5041, D5042, D5043, D5044, D5045, D5046, D5047, D5048: SK6812MINI, local-libraries:SK6812_mini_e_corners, symbol LED:SK6812MINI
- removed F1: Polyfuse, Fuse:Fuse_0603_1608Metric, symbol Device:Polyfuse
- removed FB1: FerriteBead_Small, Inductor_SMD:L_0603_1608Metric, symbol Device:FerriteBead_Small
- removed J1: USB_C_Receptacle_USB2.0, 0xLib_USB_Type-C:USB_C_Receptacle_HRO_TYPE-C-31-M-13B, symbol Connector:USB_C_Receptacle_USB2.0
- removed J102: NA_serial, local-libraries:Jack_3.5mm_PJ320E_Horizontal, symbol Connector:AudioJack4
- removed J105: NA_Conn_01x04_Female, local-libraries:PinHeader_1x04_P2.54mm_Vertical_debug, symbol Connector:Conn_01x04_Female
- removed J113: Cirque, local-libraries:FPC-SMD_FPC05012-09200-.5mm, symbol Connector:Conn_01x14_Female
- removed J3: NA_GC9A01, local-libraries:PinHeader_1x07_P2.54mm_Vertical, symbol kbd:IPS_LCD__gc9a01_240X240
- removed J4, J5010: Conn_01x05, local-libraries:PinHeader_1x05_P1.27mm_Vertical_SMD, symbol Connector_Generic:Conn_01x05
- removed J5: NA_Conn_01x02, Connector_PinHeader_1.27mm:PinHeader_1x02_P1.27mm_Vertical, symbol Connector_Generic:Conn_01x02
- removed O101: NA_OLED, local-libraries:PinHeader_1x04_P2.54mm_Vertical, symbol Connector_Generic:Conn_01x04
- removed R1, R3, R8: 1k, Resistor_SMD:R_0402_1005Metric, symbol Device:R
- removed R10, R4, R5: 5.1k, Resistor_SMD:R_0402_1005Metric, symbol Device:R
- removed R101: 5.1k, local-libraries:R_0402_1005Metric_nolabel, symbol Device:R
- removed R103, R104: 4.7k, local-libraries:R_0402_1005Metric_nolabel, symbol Device:R
- removed R11, R2, R9: 10k, Resistor_SMD:R_0402_1005Metric, symbol Device:R
- removed R5016: 330, Resistor_SMD:R_0402_1005Metric, symbol Device:R
- removed R6, R7: 27, Resistor_SMD:R_0402_1005Metric, symbol Device:R
- removed SW1: SW_Push, Button_Switch_SMD:SW_SPST_CK_KXT3, symbol Switch:SW_Push
- removed SW3002: NA_RotaryEncoder_Switch, local-libraries:RotaryEncoder_Alps_EC11E-Switch_Vertical_H20mm_roundholes, symbol Device:RotaryEncoder_Switch
- removed U1: RP2040, 0xLib_Package_DFN_QFN:QFN-56-1EP_7x7mm_P0.4mm_EP3.2x3.2mm, symbol MCU_RaspberryPi_RP2040:RP2040
- removed U2: W25Q128JVS, drawings:W25Q128JVPIQ, symbol Memory_Flash:W25Q128JVS
- removed U3: XC6210B332MR-G, Package_TO_SOT_SMD:SOT-23-5, symbol Regulator_Linear:AP2127K-3.3
- removed U4, U5005: USBLC6-2P6, Package_TO_SOT_SMD:SOT-666, symbol Power_Protection:USBLC6-2P6
- removed Y1: Crystal_GND24, Crystal:Crystal_SMD_2520-4Pin_2.5x2.0mm, symbol Device:Crystal_GND24
- added D5031, D5032, D5033, D5034, D5035, D5036, D5037, D5038, D5039, D5040, D5041, D5042, D5043, D5044, D5045, D5046: D, Diode_SMD:D_SOD-123, symbol Device:D
- added J5011: BATTERY_CONN_DEANS, local-libraries:battery_connector_THT, symbol SparkFun-Connectors:BATTERY_CONN_DEANS
- added PSW5001: SW_DPDT_x2, local-libraries:Switch_MSK-12C01-07, symbol jiran-ble:SW_DPDT
- added U5007: eliteC, local-libraries:Sparkfun_Pro_Micro, symbol elite-C:eliteC
- D112, D115: footprint local-libraries:D_SOD-323 -> Diode_SMD:D_SOD-123
Connections:
- net GND: now also J5011.-, U5007.23 (GND), U5007.3 (GND), U5007.4 (GND)
- net M_COL1: now also D5031.1 (K), D5032.1 (K), D5033.1 (K), D5034.1 (K), U5007.11 (B4)
- net M_COL2: now also D5035.1 (K), D5036.1 (K), D5037.1 (K), D5038.1 (K), U5007.12 (B5)
- net M_COL3: now also D5039.1 (K), D5040.1 (K), D5041.1 (K), D5042.1 (K), U5007.10 (E6)
- net M_COL4: now also D5043.1 (K), D5044.1 (K), U5007.9 (D7)
- net M_COL5: now also D5045.1 (K), D5046.1 (K), U5007.18 (F6)
- net M_ROW1: now also U5007.17 (F7)
- net M_ROW2: now also U5007.7 (D4)
- net M_ROW3: now also U5007.8 (C6)
- net M_ROW4: now also U5007.19 (F5)
- net at SW118.2: now also D5034.2 (A)
- net at SW109.2: now also D5041.2 (A)
- net at SW105.2: now also D5036.2 (A)
- net at SW108.2: now also D5040.2 (A)
- net at SW107.2: now also D5039.2 (A)
- net at SW102.2: now also D5032.2 (A)
- net at SW115.2: now also D5045.2 (A)
- net at SW116.2: now also D5046.2 (A)
- net at SW104.2: now also D5035.2 (A)
- net at SW119.2: now also D5038.2 (A)
- net at SW106.2: now also D5037.2 (A)
- net at SW113.2: now also D5044.2 (A)
- net at SW112.2: now also D5043.2 (A)
- net at SW101.2: now also D5031.2 (A)
- net at SW103.2: now also D5033.2 (A)
- net encoder_diode: no longer names the net of SW3001.2
- net encoder_diode: now also D5042.2 (A)
- net ~{RESET} renamed RESET
- net RESET: now also U5007.22 (RST)
- new net +5VL: U5007.21 (VCC)
- new net BAT: PSW5001.1 (A), U5007.24 (RAW)
- new net BAT_SW: J5011.+, PSW5001.2 (B)
- no-connect marks 30 -> 31
Other:
- note added: "Battery connector"
- note added: "Power switch"
- note removed: "reverse for left half"
- company: plut0nium x bastardkb x freznel -> bmolnar
- title: Dilemma -> Dilemma Light
- moved on the sheet: D112, D115, H101, H102, H104, H105, H106, H107, H108, H111, SW101, SW102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
