File: 3x5_3/dilemma.kicad_sch (KiCad schematic)
At the start: 89 parts, among them J5001 BATTERY_CONN_DEANS, J5011 BATTERY_CONN_DEANS, SW101 NA_SW_Push, SW102 NA_SW_Push, SW103 NA_SW_Push, SW104 NA_SW_Push, SW105 NA_SW_Push, SW106 NA_SW_Push, SW107 NA_SW_Push, SW108 NA_SW_Push, SW109 NA_SW_Push, SW112 NA_SW_Push, SW113 NA_SW_Push, SW114 NA_SW_Push, SW115 NA_SW_Push, SW116 NA_SW_Push, SW117 NA_SW_Push, SW118 NA_SW_Push, SW119 NA_SW_Push, SW3001 NA_SW_Push, SW5002 NA_SW_Push, SW5003 NA_SW_Push, SW5004 NA_SW_Push, SW5005 NA_SW_Push, SW5006 NA_SW_Push, SW5007 NA_SW_Push, SW5008 NA_SW_Push, SW5009 NA_SW_Push, SW5010 NA_SW_Push, SW5011 NA_SW_Push, SW5012 NA_SW_Push, SW5013 NA_SW_Push, SW5014 NA_SW_Push, SW5015 NA_SW_Push, SW5016 NA_SW_Push, SW5017 NA_SW_Push, SW5018 NA_SW_Push, SW5019 NA_SW_Push, SW5021 SW_SPST, SW5022 SW_SPST, U5001 eliteC, U5007 eliteC

Commit message: reroute
Connections:
- net BAT: now also PSW5001.1 (A); no longer PSW5001.2 (B)
- net BAT_SW: now also PSW5001.2 (B); no longer PSW5001.1 (A)
Other:
- moved on the sheet: PSW5001
Changed lines of the file:
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@@
 	)
 	(no_connect
-		(at 30.48 123.19)
+		(at 26.67 123.19)
 	)
 	(no_connect
@@
 	(global_label "BAT"
 		(shape input)
-		(at 40.64 120.65 0)
+		(at 26.67 118.11 180)
 		(effects
 			(font
 				(size 1.27 1.27)
 			)
-			(justify left)
+			(justify right)
 		)
 		(property "Intersheetrefs" "${INTERSHEET_REFS}"
-			(at -82.55 -10.16 0)
+			(at 149.86 248.92 0)
 			(effects
 				(font
@@
 	(global_label "BAT_SW"
 		(shape input)
-		(at 30.48 118.11 180)
+		(at 36.83 120.65 0)
 		(effects
 			(font
 				(size 1.27 1.27)
 			)
-			(justify right)
+			(justify left)
 		)
 		(property "Intersheetrefs" "${INTERSHEET_REFS}"
-			(at 153.67 248.92 0)
+			(at -86.36 -10.16 0)
 			(effects
 				(font
@@
 	(symbol
 		(lib_id "jiran-ble:SW_DPDT")
-		(at 34.29 120.65 0)
+		(at 30.48 120.65 0)
 		(mirror y)
 		(unit 1)
@@
 		(dnp no)
 		(property "Reference" "PSW5001"
-			(at 35.56 112.395 0)
+			(at 31.75 112.395 0)
 			(effects
 				(font
@@
 		)
 		(property "Value" "SW_DPDT_x2"
-			(at 35.56 114.935 0)
+			(at 31.75 114.935 0)
 			(effects
 				(font
@@
 		)
 		(property "Footprint" "local-libraries:Switch_MSK-12C01-07"
-			(at 33.655 113.03 0)
+			(at 29.845 113.03 0)
 			(effects
 				(font
@@
 		)
 		(property "Datasheet" ""
-			(at 33.655 113.03 0)
+			(at 29.845 113.03 0)
 			(effects
 				(font
@@
 		)
 		(property "Description" ""
-			(at 34.29 120.65 0)
+			(at 30.48 120.65 0)
 			(effects
 				(font
@@
 		)
 		(property "LCSC" "C431540"
-			(at 34.29 120.65 0)
+			(at 30.48 120.65 0)
 			(effects
 				(font
